File: hardware/stm32_bob_v2.brd (EAGLE design)
At the start: 108.9 x 72.1 mm, 49 parts, among them U1 F3_DISCOVERY, U2 LSF0108, U3 INA827, U4 INA827

Commit message: changed io to avoid pins used on development board
Connections:
- net PA14_5 renamed PB8_5
- net PA15_5 renamed PB9_5
- net PE11_5 renamed PA9_5
- net PE13_5 renamed PA10_5
- net PE14_5 renamed PB0_5
- net PE9_5 renamed PA8_5
- net PA0: no longer R4.1
- net PA1: now also R4.1; no longer U$1.5
- net PA10: now also R8.1, U2.5
- net PA11: no longer U$1.21
- net PA12: no longer U$1.22
- net PA14: no longer R10.2, U2.7
- net PA15: now also U$1.21; no longer R11.2, U2.8
- net PA5: no longer U$1.9
- net PA6: no longer U$1.11
- net PA7: no longer U$1.12
- net PA8: now also R6.1, U2.3
- net PA9: now also R7.1, U2.4
- net PB0: now also R9.1, U2.6
- net PB10: now also U$1.24
- net PB11: now also U$1.22
- net PB13: now also U$1.9
- net PB14: now also U$1.11
- net PB15: now also U$1.12
- net PB2: now also U$1.5
- net PB3: no longer U$1.17
- net PB8: now also R10.2, U2.7
- net PB9: now also R11.2, U2.8
- net PC12: now also U$1.17
- net PE11: no longer R7.1, U2.4
- net PE13: no longer R8.1, U2.5
- net PE14: no longer R9.1, U2.6
- net PE15: no longer U$1.24
- net PE9: no longer R6.1, U2.3
Routing:
- net PA0: track 93.5 -> 0.00 mm, vias 4 -> 0
- net PA1: track 10.7 -> 95.3 mm, vias 0 -> 2
- net PA12: track 71.7 -> 0.00 mm, vias 3 -> 0
- net PA11: track 71.3 -> 0.00 mm, vias 3 -> 0
- net PC12: track 0.00 -> 69.4 mm, vias 0 -> 4
- net PB3: track 68.2 -> 0.00 mm, vias 4 -> 0
- net PA15: track 27.2 -> 91.3 mm, vias 1 -> 10
- net PB10: track 0.00 -> 53.9 mm, vias 0 -> 7
- net PE9: track 52.0 -> 0.00 mm, vias 2 -> 0
- net PB0: track 0.00 -> 47.1 mm, vias 0 -> 2
- net PE11: track 46.3 -> 0.00 mm, vias 4 -> 0
- net PB9: track 0.00 -> 46.3 mm, vias 0 -> 3
- net PB8: track 0.00 -> 46.2 mm, vias 0 -> 3
- net PE13: track 42.7 -> 0.00 mm, vias 2 -> 0
- net PE14: track 37.8 -> 0.00 mm
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Other:
- board text added: "3V 3V 5V 5V PB2 PA2 PA3 PF4 PB13 GND"
- board text added: "PA15 PB11 PB1 PB10 PB12 PC11_5 PC10_5 PB9_5 PB8_5 GND"
- board text added: "PB0_5 PA10_5 PA9_5 PA8_5 AIN1_N AIN1_P AIN2_N AIN2_P REF_EXT GND"
- board text added: "PB14 PB15 PC6 PC7 PC8 PC9 PC12 PB4 PB5 GND"
- board text removed: "3.3V 3.3V 5V 5V PA1 PA2 PA3 PF4 PA5 GND"
- board text removed: "PA11 PA12 PB1 PE15 PB12 PC11_5 PC10_5 PA15_5 PA14_5 GND"
- board text removed: "PA6 PA7 PC6 PC7 PC8 PC9 PB3 PB4 PB5 GND"
- board text removed: "PE14_5 PE13_5 PE11_5 PE9_5 AIN1_N AIN1_P AIN2_N AIN2_P REF_EXT GND"
